Commit message: use robotiq 2f 85

File: kortex_description/robots/kinova_gen3.urdf (robot description, URDF)
Before this commit: robot kinova, 11 links, 10 joints
Links:
- removed link panda_hand
- removed link panda_leftfinger
- removed link panda_rightfinger
- added link end_effector_link, mass 0
- added link robotiq_2f_85_base, mass 0.1; collision mesh filename=package://kortex_description/meshes/robotiq-2f-base.stl scale=0.001 0.001 0.001; visual mesh filename=package://kortex_description/meshes/robotiq-2f-base.stl scale=0.001 0.001 0.001
- added link robotiq_2f_85_left_coupler, mass 0.1; collision mesh filename=package://kortex_description/meshes/robotiq-2f-coupler.stl scale=0.001 0.001 0.001; visual mesh filename=package://kortex_description/meshes/robotiq-2f-coupler.stl scale=0.001 0.001 0.001
- added link robotiq_2f_85_left_driver, mass 0.1; collision mesh filename=package://kortex_description/meshes/robotiq-2f-driver.stl scale=0.001 0.001 0.001; visual mesh filename=package://kortex_description/meshes/robotiq-2f-driver.stl scale=0.001 0.001 0.001
- added link robotiq_2f_85_left_follower, mass 0.1; collision mesh filename=package://kortex_description/meshes/robotiq-2f-follower.stl scale=0.001 0.001 0.001; visual mesh filename=package://kortex_description/meshes/robotiq-2f-follower.stl scale=0.001 0.001 0.001
- added link robotiq_2f_85_left_pad, mass 0.1; collision mesh filename=package://kortex_description/meshes/robotiq-2f-pad.stl name=b scale=0.001 0.001 0.001; visual mesh filename=package://kortex_description/meshes/robotiq-2f-pad.stl name=a scale=0.0001 0.0001 0.0001
- added link robotiq_2f_85_left_spring_link, mass 0.1; collision mesh filename=package://kortex_description/meshes/robotiq-2f-spring_link.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 scale=0.001 0.001 0.001; visual mesh filename=package://kortex_description/meshes/robotiq-2f-spring_link.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 scale=0.001 0.001 0.001
- added link robotiq_2f_85_right_coupler, mass 0.1; collision mesh filename=package://kortex_description/meshes/robotiq-2f-coupler.stl scale=0.001 0.001 0.001; visual mesh filename=package://kortex_description/meshes/robotiq-2f-coupler.stl scale=0.001 0.001 0.001
- added link robotiq_2f_85_right_driver, mass 0.1; collision mesh filename=package://kortex_description/meshes/robotiq-2f-driver.stl scale=0.001 0.001 0.001; visual mesh filename=package://kortex_description/meshes/robotiq-2f-driver.stl scale=0.001 0.001 0.001
- added link robotiq_2f_85_right_follower, mass 0.1; collision mesh filename=package://kortex_description/meshes/robotiq-2f-follower.stl scale=0.001 0.001 0.001; visual mesh filename=package://kortex_description/meshes/robotiq-2f-follower.stl scale=0.001 0.001 0.001
- added link robotiq_2f_85_right_pad, mass 0.1; collision mesh filename=package://kortex_description/meshes/robotiq-2f-pad.stl scale=0.001 0.001 0.001; visual mesh filename=package://kortex_description/meshes/robotiq-2f-pad.stl scale=0.0001 0.0001 0.0001
- added link robotiq_2f_85_right_spring_link, mass 0.1; collision mesh filename=package://kortex_description/meshes/robotiq-2f-spring_link.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 scale=0.001 0.001 0.001; visual mesh filename=package://kortex_description/meshes/robotiq-2f-spring_link.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 scale=0.001 0.001 0.001
Joints:
- removed joint panda_finger_joint1
- removed joint panda_finger_joint2
- removed joint panda_hand_joint
- added joint base_link_robotiq_2f_85_base_joint: type fixed, parent end_effector_link, child robotiq_2f_85_base, origin xyz=0 0 0 rpy=0 0 0
- added joint end_effector: type fixed, parent bracelet_link, child end_effector_link, origin xyz=0 0 -0.061525 rpy=-3.1415 0 1.57, axis 0 0 0
- added joint robotiq_2f_85_left_coupler_joint: type fixed, parent robotiq_2f_85_left_driver, child robotiq_2f_85_left_coupler, origin xyz=0 0.0315 -0.0041 rpy=0 0 0
- added joint robotiq_2f_85_left_driver_joint: type fixed, parent robotiq_2f_85_base, child robotiq_2f_85_left_driver, origin xyz=0 -0.0306011 0.054904 rpy=0 0 3.141592653589793, axis 1 0 0, limit lower=0.0 upper=0.834 effort=176 velocity=1.91986177778, mimic joint=robotiq_2f_85_right_driver_joint multiplier=1
- added joint robotiq_2f_85_left_follower_joint: type fixed, parent robotiq_2f_85_left_coupler, child robotiq_2f_85_left_follower, origin xyz=0 0.0061 0.0471 rpy=0 0 0, axis 1 0 0, limit lower=-2.96705911111 upper=2.96705911111 effort=176 velocity=1.91986177778, mimic joint=robotiq_2f_85_right_driver_joint multiplier=-1
- added joint robotiq_2f_85_left_pad_joint: type revolute, parent robotiq_2f_85_left_follower, child robotiq_2f_85_left_pad
- added joint robotiq_2f_85_left_spring_link_joint: type fixed, parent robotiq_2f_85_base, child robotiq_2f_85_left_spring_link, origin xyz=0 -0.012 0.0614 rpy=0 0 3.141592653589793, axis 1 0 0, limit lower=-2.96705911111 upper=2.96705911111 effort=176 velocity=1.91986177778, mimic joint=robotiq_2f_85_right_driver_joint multiplier=1
- added joint robotiq_2f_85_right_coupler_joint: type fixed, parent robotiq_2f_85_right_driver, child robotiq_2f_85_right_coupler, origin xyz=0 0.0315 -0.0041 rpy=0 0 0
- added joint robotiq_2f_85_right_driver_joint: type fixed, parent robotiq_2f_85_base, child robotiq_2f_85_right_driver, origin xyz=0 0.0306011 0.054904 rpy=0 0 0, axis 1 0 0, limit lower=0.0 upper=0.834 effort=60 velocity=1.91986177778
- added joint robotiq_2f_85_right_follower_joint: type fixed, parent robotiq_2f_85_right_coupler, child robotiq_2f_85_right_follower, origin xyz=0 0.0061 0.0471 rpy=0 0 0, axis 1 0 0, limit lower=-2.96705911111 upper=2.96705911111 effort=176 velocity=1.91986177778, mimic joint=robotiq_2f_85_right_driver_joint multiplier=-1
- added joint robotiq_2f_85_right_pad_joint: type revolute, parent robotiq_2f_85_right_follower, child robotiq_2f_85_right_pad
- added joint robotiq_2f_85_right_spring_link_joint: type fixed, parent robotiq_2f_85_base, child robotiq_2f_85_right_spring_link, origin xyz=0 0.012 0.0614 rpy=0 0 0, axis 1 0 0, limit lower=-2.96705911111 upper=2.96705911111 effort=176 velocity=1.91986177778, mimic joint=robotiq_2f_85_right_driver_joint multiplier=1
